File: hardware/Adaptateur/Adaptateur.kicad_sch (KiCad schematic)
At the start: 17 parts, among them J1 USB_B, SW1 SW_Push_SPDT, U1 FT231XS, U2 XBEE-3-TH, U3 NCP1117-3.3_SOT223

Commit message: Commit avant nouveau projet
Parts:
- removed SW1: SW_Push_SPDT, Button_Switch_THT:SW_PUSH_6mm_H5mm, symbol Switch:SW_Push_SPDT
- added H1, H2, H3, H4: MountingHole_Pad, MountingHole:MountingHole_3.2mm_M3_DIN965_Pad, symbol Mechanical:MountingHole_Pad
- added R3: 10K, Resistor_SMD:R_1206_3216Metric, symbol Device:R
- added SW1: SW_DPST_x2, Button_Switch_THT:SW_PUSH_6mm_H4.3mm, symbol Switch:SW_DPST_x2
Connections:
- net +3.3V: now also R3.2
- net GND: now also H1.1, H2.1, H3.1, H4.1, SW1.2 (B)
- net at U2.5 (~{RESET}): now also R3.1, SW1.1 (A)
