File: laas/Multiprise pilotée/DC_supplies.kicad_sch (KiCad schematic)
At the start: 18 parts, among them J7 Conn_02x06_Odd_Even, Q1 DMN2020LSN-7, Q2 DMN2020LSN-7, Q3 SSM3J355R,LF, Q4 DMN2020LSN-7, Q5 DMN2020LSN-7, Q6 SSM3J355R,LF, Q7 DMN2020LSN-7, Q8 DMN2020LSN-7, U2 74HC595, U4 TC4469, U5 TC4469

Commit message: Sauvegarde du travail en cours
Parts:
- added U6: TDA7391PD, footprints:SO_91PDTR_STM, symbol Multiprise pilotée:TDA7391PD
- added U7: 74AHC1G08, Package_TO_SOT_SMD:SOT-23-5, symbol 74xGxx:74AHC1G08
- J7: footprint (none) -> Connector_JAE:JAE_LY20-14P-DT1_2x07_P2.00mm_Vertical
Connections:
- net +5V: now also U6.16 (VCC2), U6.5 (VCC1), U7.5 (VCC)
- net GND: now also C3.2, U6.1 (P-GND), U6.10 (P-GND), U6.11 (P-GND), U6.12 (S-GND), U6.14 (IN-), U6.20 (P-GND), U7.3 (GND); no longer J7.12 (Pin_12), U2.10 (~{SRCLR})
- net PWR_+5V: now also Q3.3 (D), Q7.3 (D)
- net PWR_-5V: now also Q6.3 (D), Q8.3 (D)
- net SCLK: now also U7.1; no longer U2.12 (RCLK)
- net ~{RESET_IO}: now also U2.10 (~{SRCLR}); no longer U2.11 (SRCLK)
- net PWM_PWR_VAR: now reaches R2.1
- net at R2.2: now also C3.1, U6.15 (IN+)
- net DRV_+5V_A: now reaches U2.4 (QE)
- net DRV_+5V_A: now also U5.1 (1A)
- net DRV_+5V_B: now reaches U2.5 (QF)
- net DRV_+5V_B: now also U5.3 (2A)
- net DRV_-5V_A: now reaches U2.6 (QG)
- net DRV_-5V_A: now also U5.5 (3A)
- net DRV_-5V_B: now reaches U2.7 (QH)
- net DRV_-5V_B: now also U5.8 (4A)
- net PWR_VAR renamed PWR_VAR_POS
- net PWR_VAR_POS: now also U6.2 (OUT+)
- new net: U2.11 (SRCLK), U7.4
- new net CS_PWR_DC: U7.2
- new net LATCH: U2.12 (RCLK)
- new net PWR_VAR_NEG: J7.12 (Pin_12), U6.19 (OUT-)
- no-connect marks 5 -> 2
Other:
- moved on the sheet: C3, Q3, Q6, Q7, Q8, R2, U2, U4, U5

Commit message: Commit de propreté
Parts:
- added C4: 33µF, Capacitor_SMD:C_1206_3216Metric, symbol Device:C
- added R7: 56K, Resistor_SMD:R_1206_3216Metric, symbol Device:R
- J7: footprint Connector_JAE:JAE_LY20-14P-DT1_2x07_P2.00mm_Vertical -> Borniers:M80-85312YY; symbol Connector_Generic:Conn_02x06_Odd_Even -> Connector_Generic:Conn_02x06_Top_Bottom
Connections:
- net +3V3: now also J7.7 (Pin_7), J7.8 (Pin_8), J7.9 (Pin_9); no longer J7.2 (Pin_2), J7.4 (Pin_4), J7.6 (Pin_6)
- net +5V: now also J7.10 (Pin_10); no longer J7.8 (Pin_8)
- net GND: now also C4.2, R7.1
- net PWR_+5V: now also J7.5 (Pin_5); no longer J7.9 (Pin_9)
- net PWR_-5V: now also J7.11 (Pin_11); no longer J7.10 (Pin_10)
- net PWR_3V3_2: now also J7.2 (Pin_2); no longer J7.3 (Pin_3)
- net PWR_3V3_3: now also J7.3 (Pin_3); no longer J7.5 (Pin_5)
- net PWR_5V_1: now also J7.4 (Pin_4); no longer J7.7 (Pin_7)
- net PWR_VAR_POS: now also J7.6 (Pin_6); no longer J7.11 (Pin_11)
- net at U6.8 (SYNC): now also R7.2
- net at U6.9 (MUTE): now also C4.1
- no-connect marks 2 -> 3
Other:
- moved on the sheet: C3, R2
Changed lines of the file:
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@@
   (junction (at 127 60.96) (diameter 0) (color 0 0 0 0)
   )
+  (junction (at 194.31 130.81) (diameter 0) (color 0 0 0 0)
+  )
   (junction (at 223.52 130.81) (diameter 0) (color 0 0 0 0)
   )
@@
   (junction (at 251.46 64.77) (diameter 0) (color 0 0 0 0)
   )
+  (junction (at 201.93 130.81) (diameter 0) (color 0 0 0 0)
+  )
   (junction (at 138.43 156.21) (diameter 0) (color 0 0 0 0)
   )
   (junction (at 200.66 49.53) (diameter 0) (color 0 0 0 0)
   )
-  (junction (at 187.96 104.14) (diameter 0) (color 0 0 0 0)
+  (junction (at 167.64 104.14) (diameter 0) (color 0 0 0 0)
   )
   (no_connect (at 105.41 62.23))
+  (no_connect (at 204.47 115.57))
   (no_connect (at 232.41 114.3))
   (wire (pts (xy 127 54.61) (xy 129.54 54.61))
@@
     (stroke (width 0) (type default))
   )
+  (wire (pts (xy 180.34 127) (xy 180.34 130.81))
+    (stroke (width 0) (type default))
+  )
   (wire (pts (xy 152.4 40.64) (xy 166.37 40.64))
     (stroke (width 0) (type default))
@@
     (stroke (width 0) (type default))
   )
+  (wire (pts (xy 201.93 130.81) (xy 194.31 130.81))
+    (stroke (width 0) (type default))
+  )
   (wire (pts (xy 63.5 163.83) (xy 63.5 160.02))
     (stroke (width 0) (type default))
@@
     (stroke (width 0) (type default))
   )
-  (wire (pts (xy 184.15 104.14) (xy 187.96 104.14))
+  (wire (pts (xy 163.83 104.14) (xy 167.64 104.14))
     (stroke (width 0) (type default))
   )
@@
     (stroke (width 0) (type default))
   )
-  (wire (pts (xy 187.96 111.76) (xy 187.96 114.3))
-    (stroke (width 0) (type default))
-  )
-  (wire (pts (xy 187.96 104.14) (xy 204.47 104.14))
+  (wire (pts (xy 167.64 111.76) (xy 167.64 114.3))
+    (stroke (width 0) (type default))
+  )
+  (wire (pts (xy 167.64 104.14) (xy 204.47 104.14))
     (stroke (width 0) (type default))
   )
@@
     (stroke (width 0) (type default))
   )
+  (wire (pts (xy 194.31 118.11) (xy 194.31 119.38))
+    (stroke (width 0) (type default))
+  )
   (wire (pts (xy 116.84 105.41) (xy 119.38 105.41))
     (stroke (width 0) (type default))
@@
     (stroke (width 0) (type default))
   )
+  (wire (pts (xy 180.34 113.03) (xy 180.34 119.38))
+    (stroke (width 0) (type default))
+  )
   (wire (pts (xy 82.55 54.61) (xy 85.09 54.61))
     (stroke (width 0) (type default))
@@
     (stroke (width 0) (type default))
   )
+  (wire (pts (xy 204.47 118.11) (xy 194.31 118.11))
+    (stroke (width 0) (type default))
+  )
+  (wire (pts (xy 194.31 127) (xy 194.31 130.81))
+    (stroke (width 0) (type default))
+  )
   (wire (pts (xy 252.73 49.53) (xy 252.73 59.69))
     (stroke (width 0) (type default))
   )
-  (wire (pts (xy 172.72 104.14) (xy 176.53 104.14))
+  (wire (pts (xy 152.4 104.14) (xy 156.21 104.14))
     (stroke (width 0) (type default))
   )
@@
     (stroke (width 0) (type default))
   )
+  (wire (pts (xy 194.31 130.81) (xy 180.34 130.81))
+    (stroke (width 0) (type default))
+  )
   (wire (pts (xy 53.34 168.91) (xy 55.88 168.91))
     (stroke (width 0) (type default))
@@
   )
   (wire (pts (xy 105.41 44.45) (xy 123.19 44.45))
+    (stroke (width 0) (type default))
+  )
+  (wire (pts (xy 204.47 113.03) (xy 180.34 113.03))
     (stroke (width 0) (type default))
   )
@@
     (effects (font (size 1.27 1.27)) (justify left bottom))
   )
-  (hierarchical_label "PWM_PWR_VAR" (shape input) (at 172.72 104.14 180) (fields_autoplaced)
+  (hierarchical_label "PWM_PWR_VAR" (shape input) (at 152.4 104.14 180) (fields_autoplaced)
     (effects (font (size 1.27 1.27)) (justify right))
   )
@@
   (hierarchical_label "MOSI" (shape input) (at 76.2 39.37 180) (fields_autoplaced)
     (effects (font (size 1.27 1.27)) (justify right))
+  )
+  (symbol (lib_id "Device:R") (at 194.31 123.19 180) (unit 1)
+    (in_bom yes) (on_board yes) (dnp no) (fields_autoplaced)
+    (property "Reference" "R7" (at 196.85 121.92 0)
+      (effects (font (size 1.27 1.27)) (justify right))
+    )
+    (property "Value" "56K" (at 196.85 124.46 0)
+      (effects (font (size 1.27 1.27)) (justify right))
+    )
+    (property "Footprint" "Resistor_SMD:R_1206_3216Metric" (at 196.088 123.19 90)
+      (effects (font (size 1.27 1.27)) hide)
+    )
+    (property "Datasheet" "~" (at 194.31 123.19 0)
+      (effects (font (size 1.27 1.27)) hide)
+    )
+    (pin "2")
+    (pin "1")
+    (instances
+      (project "Multiprise pilotée"
+        (path "/ad17dd83-c10a-426e-803d-3b2dda0cc379/7b0b359f-83f5-4bfc-867e-e59ab7e7da3c"
+          (reference "R7") (unit 1)
+        )
+      )
+    )
   )
   (symbol (lib_id "power:GND") (at 214.63 69.85 0) (unit 1)
@@
     )
   )
-  (symbol (lib_id "Device:R") (at 180.34 104.14 90) (unit 1)
-    (in_bom yes) (on_board yes) (dnp no) (fields_autoplaced)
-    (property "Reference" "R2" (at 180.34 97.79 90)
-      (effects (font (size 1.27 1.27)))
-    )
-    (property "Value" "10R" (at 180.34 100.33 90)
-      (effects (font (size 1.27 1.27)))
-    )
-    (property "Footprint" "Resistor_SMD:R_1206_3216Metric" (at 180.34 105.918 90)
-      (effects (font (size 1.27 1.27)) hide)
-    )
-    (property "Datasheet" "~" (at 180.34 104.14 0)
+  (symbol (lib_id "Device:R") (at 160.02 104.14 90) (unit 1)
+    (in_bom yes) (on_board yes) (dnp no) (fields_autoplaced)
+    (property "Reference" "R2" (at 160.02 97.79 90)
+      (effects (font (size 1.27 1.27)))
+    )
+    (property "Value" "10R" (at 160.02 100.33 90)
+      (effects (font (size 1.27 1.27)))
+    )
+    (property "Footprint" "Resistor_SMD:R_1206_3216Metric" (at 160.02 105.918 90)
+      (effects (font (size 1.27 1.27)) hide)
+    )
+    (property "Datasheet" "~" (at 160.02 104.14 0)
       (effects (font (size 1.27 1.27)) hide)
     )
@@
     )
   )
-  (symbol (lib_id "power:GND") (at 187.96 114.3 0) (unit 1)
-    (in_bom yes) (on_board yes) (dnp no) (fields_autoplaced)
-    (property "Reference" "#PWR025" (at 187.96 120.65 0)
-      (effects (font (size 1.27 1.27)) hide)
-    )
-    (property "Value" "GND" (at 187.96 119.38 0)
-      (effects (font (size 1.27 1.27)))
-    )
-    (property "Footprint" "" (at 187.96 114.3 0)
-      (effects (font (size 1.27 1.27)) hide)
-    )
-    (property "Datasheet" "" (at 187.96 114.3 0)
+  (symbol (lib_id "power:GND") (at 167.64 114.3 0) (unit 1)
+    (in_bom yes) (on_board yes) (dnp no) (fields_autoplaced)
+    (property "Reference" "#PWR025" (at 167.64 120.65 0)
+      (effects (font (size 1.27 1.27)) hide)
+    )
+    (property "Value" "GND" (at 167.64 119.38 0)
+      (effects (font (size 1.27 1.27)))
+    )
+    (property "Footprint" "" (at 167.64 114.3 0)
+      (effects (font (size 1.27 1.27)) hide)
+    )
+    (property "Datasheet" "" (at 167.64 114.3 0)
       (effects (font (size 1.27 1.27)) hide)
     )
@@
     )
   )
-  (symbol (lib_id "Connector_Generic:Conn_02x06_Odd_Even") (at 127 161.29 0) (unit 1)
+  (symbol (lib_id "Connector_Generic:Conn_02x06_Top_Bottom") (at 127 161.29 0) (unit 1)
     (in_bom yes) (on_board yes) (dnp no)
     (property "Reference" "J7" (at 128.27 152.4 0)
@@
       (effects (font (size 1.27 1.27)) hide)
     )
-    (property "Footprint" "Connector_JAE:JAE_LY20-14P-DT1_2x07_P2.00mm_Vertical" (at 127 161.29 0)
+    (property "Footprint" "Borniers:M80-85312YY" (at 127 161.29 0)
       (effects (font (size 1.27 1.27)) hide)
     )
@@
     )
   )
+  (symbol (lib_id "Device:C") (at 180.34 123.19 0) (unit 1)
+    (in_bom yes) (on_board yes) (dnp no) (fields_autoplaced)
+    (property "Reference" "C4" (at 184.15 121.92 0)
+      (effects (font (size 1.27 1.27)) (justify left))
+    )
+    (property "Value" "33µF" (at 184.15 124.46 0)
+      (effects (font (size 1.27 1.27)) (justify left))
+    )
+    (property "Footprint" "Capacitor_SMD:C_1206_3216Metric" (at 181.3052 127 0)
+      (effects (font (size 1.27 1.27)) hide)
+    )
+    (property "Datasheet" "~" (at 180.34 123.19 0)
+      (effects (font (size 1.27 1.27)) hide)
+    )
+    (pin "1")
+    (pin "2")
+    (instances
+      (project "Multiprise pilotée"
+        (path "/ad17dd83-c10a-426e-803d-3b2dda0cc379/7b0b359f-83f5-4bfc-867e-e59ab7e7da3c"
+          (reference "C4") (unit 1)
+        )
+      )
+    )
+  )
   (symbol (lib_id "Device:Q_PMOS_GSD") (at 237.49 41.91 0) (mirror x) (unit 1)
     (in_bom yes) (on_board yes) (dnp no)
@@
     )
   )
-  (symbol (lib_id "Device:C") (at 187.96 107.95 0) (unit 1)
-    (in_bom yes) (on_board yes) (dnp no) (fields_autoplaced)
-    (property "Reference" "C3" (at 191.77 106.68 0)
-      (effects (font (size 1.27 1.27)) (justify left))
-    )
-    (property "Value" "100nF" (at 191.77 109.22 0)
-      (effects (font (size 1.27 1.27)) (justify left))
-    )
-    (property "Footprint" "Capacitor_SMD:C_1206_3216Metric" (at 188.9252 111.76 0)
-      (effects (font (size 1.27 1.27)) hide)
-    )
-    (property "Datasheet" "~" (at 187.96 107.95 0)
-      (effects (font (size 1.27 1.27)) hide)
-    )
+  (symbol (lib_id "Device:C") (at 167.64 107.95 0) (unit 1)
+    (in_bom yes) (on_board yes) (dnp no) (fields_autoplaced)
+    (property "Reference" "C3" (at 171.45 106.68 0)
+      (effects (font (size 1.27 1.27)) (justify left))
+    )
+    (property "Value" "100nF" (at 171.45 109.22 0)
+      (effects (font (size 1.27 1.27)) (justify left))
+    )
+    (property "Footprint" "Capacitor_SMD:C_1206_3216Metric" (at 168.6052 111.76 0)
+      (effects (font (size 1.27 1.27)) hide)
+    )
+    (property "Datasheet" "~" (at 167.64 107.95 0)
+      (effects (font (size 1.27 1.27)) hide)
+    )

Commit message: Ajout du projet asservissement de balle en python
Parts:
- C3: value 100nF -> 10µF
- R2: value 10R -> 1.5K
Other:
- note added: "R=1.5K C=10µF Fc = 1/2piRC = 10Hz"
Changed lines of the file:
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@@
     (stroke (width 0) (type default))
+  )
+  (polyline (pts (xy 154.94 113.03) (xy 154.94 95.25))
+    (stroke (width 0) (type dash))
   )
   (wire (pts (xy 127 100.33) (xy 127 96.52))
@@
     (stroke (width 0) (type default))
   )
+  (polyline (pts (xy 179.07 95.25) (xy 179.07 113.03))
+    (stroke (width 0) (type dash))
+  )
   (wire (pts (xy 240.03 33.02) (xy 251.46 33.02))
     (stroke (width 0) (type default))
@@
     (stroke (width 0) (type default))
   )
+  (polyline (pts (xy 179.07 113.03) (xy 154.94 113.03))
+    (stroke (width 0) (type dash))
+  )
   (wire (pts (xy 200.66 43.18) (xy 203.2 43.18))
     (stroke (width 0) (type default))
@@
   (wire (pts (xy 262.89 46.99) (xy 262.89 49.53))
     (stroke (width 0) (type default))
+  )
+  (polyline (pts (xy 154.94 95.25) (xy 179.07 95.25))
+    (stroke (width 0) (type dash))
+  )
+  (text "R=1.5K\nC=10µF\nFc = 1/2piRC = 10Hz" (at 181.61 99.06 0)
+    (effects (font (size 1.27 1.27)) (justify left bottom))
   )
   (label "DRV_-5V_B" (at 189.23 59.69 0) (fields_autoplaced)
@@
       (effects (font (size 1.27 1.27)))
     )
-    (property "Value" "10R" (at 160.02 100.33 90)
+    (property "Value" "1.5K" (at 160.02 100.33 90)
       (effects (font (size 1.27 1.27)))
     )
@@
       (effects (font (size 1.27 1.27)) (justify left))
     )
-    (property "Value" "100nF" (at 171.45 109.22 0)
-      (effects (font (size 1.27 1.27)) (justify left))
-    )
+    (property "Value" "10µF" (at 171.45 109.22 0)
+      (effects (font (size 1.27 1.27)) (justify left))
+    )
