File: laas/Multiprise pilotée/Multiprise pilotée.kicad_pcb (KiCad board)
At the start: 2 copper layers, 4 parts, among them K1 Relay_DPDT, Q1 Q_NMOS_DGS

Commit message: Sauvegarde du travail en cours
Parts:
- added C1: 100µF, Capacitor_THT:CP_Radial_D6.3mm_P2.50mm, F.Cu at (189.2, 112.5)
- added C2: 1µF, Capacitor_SMD:C_1206_3216Metric, F.Cu at (165.5, 119.0)
- added C3: 100nF, Capacitor_SMD:C_1206_3216Metric, F.Cu at (206.9, 76.4)
- added J1: Conn_01x03, Connector_Wago:Wago_734-133_1x03_P3.50mm_Vertical, F.Cu at (166.5, 101.3)
- added J2: Conn_01x02, Connector_Wuerth:Wuerth_WR-WTB_64800211622_1x02_P1.50mm_Vertical, F.Cu at (174.0, 124.5)
- added J3: Conn_01x02, Connector_Wago:Wago_734-132_1x02_P3.50mm_Vertical, F.Cu at (155.0, 111.9)
- added J4: Conn_01x02, Connector_Wago:Wago_734-132_1x02_P3.50mm_Vertical, F.Cu at (155.0, 122.5)
- added J5: Conn_01x02, Connector_Wago:Wago_734-132_1x02_P3.50mm_Vertical, F.Cu at (155.0, 133.0)
- added J6: Conn_01x03, Connector_Wago:Wago_734-133_1x03_P3.50mm_Vertical, F.Cu at (166.5, 111.9)
- added J7: Conn_02x06_Odd_Even, Connector_JAE:JAE_LY20-14P-DT1_2x07_P2.00mm_Vertical, F.Cu at (219.7, 64.2)
- added K2: Omron Relay, Relay_THT:Relay_DPDT_Omron_G2RL-2, F.Cu at (112.1, 99.4)
- added K3: Omron Relay, Relay_THT:Relay_DPDT_Omron_G2RL-2, F.Cu at (126.2, 99.4)
- added K4: Omron Relay, Relay_THT:Relay_DPDT_Omron_G2RL-2, F.Cu at (140.4, 99.4)
- added PS2: MPM-45, Multiprise pilotée:Converter_ACDC_MeanWell_MPM-45-xx_THT, F.Cu at (114.7, 48.4)
- added Q2: DMN2020LSN-7, Package_TO_SOT_SMD:SC-59, F.Cu at (201.6, 44.5)
- added Q3: SSM3J355R,LF, Package_TO_SOT_SMD:SOT-23, F.Cu at (232.4, 63.6)
- added Q4: DMN2020LSN-7, Package_TO_SOT_SMD:SC-59, F.Cu at (201.6, 49.1)
- added Q5: DMN2020LSN-7, Package_TO_SOT_SMD:SC-59, F.Cu at (201.6, 53.8)
- added Q6: SSM3J355R,LF, Package_TO_SOT_SMD:SOT-23, F.Cu at (232.4, 68.1)
- added Q7: DMN2020LSN-7, Package_TO_SOT_SMD:SC-59, F.Cu at (201.6, 58.4)
- added Q8: DMN2020LSN-7, Package_TO_SOT_SMD:SC-59, F.Cu at (201.6, 63.1)
- added R2: 10R, Resistor_SMD:R_1206_3216Metric, F.Cu at (227.1, 63.0)
- added R3: 10R, Resistor_SMD:R_1206_3216Metric, F.Cu at (227.1, 66.3)
- added R4: 10R, Resistor_SMD:R_1206_3216Metric, F.Cu at (227.1, 69.6)
- added R5: 10R, Resistor_SMD:R_1206_3216Metric, F.Cu at (227.1, 72.9)
- added R6: 10R, Resistor_SMD:R_1206_3216Metric, F.Cu at (227.1, 76.2)
- added U1: MAX4820xUP, Package_SO:TSSOP-20-1EP_4.4x6.5mm_P0.65mm_EP2.15x3.35mm, F.Cu at (182.0, 112.5)
- added U2: 74HC595, Package_SO:SOIC-16_3.9x9.9mm_P1.27mm, F.Cu at (208.3, 69.0)
- added U3: TPS75933KC, Package_TO_SOT_SMD:TO-263-5_TabPin6, F.Cu at (188.3, 102.3)
- added U4: TC4469, Package_SO:SOIC-14W_7.5x9mm_P1.27mm, F.Cu at (210.5, 47.4)
- added U5: TC4469, Package_SO:SOIC-14W_7.5x9mm_P1.27mm, F.Cu at (210.5, 58.0)
- added U6: TDA7391PD, footprints:SO_91PDTR_STM, F.Cu at (225.5, 51.8)
- added U7: 74AHC1G08, Package_TO_SOT_SMD:SOT-23-5, F.Cu at (208.4, 85.4)
- added U8: MOUDLE-SEEEDUINO-XIAO, XIAO_PCB:MOUDLE14P-SMD-2.54-21X17.8MM, F.Cu at (60.5, 154.0)
- K1: value Relay_DPDT -> Omron Relay
- Q1: value Q_NMOS_DGS -> DMN2020LSN-7
- R1: value R -> 1K
Connections:
- K1 pad 11: unconnected-(K1-Pad11) -> LINE
- K1 pad 14: unconnected-(K1-Pad14) -> Net-(J2-Pin_1)
- K1 pad 21: unconnected-(K1-Pad21) -> NEUT
- K1 pad 24: unconnected-(K1-Pad24) -> Net-(J2-Pin_2)
- K1 pad A1: Net-(D1-A) -> +5V
- K1 pad A2: Net-(D1-K) -> /Power supply and relays/Relay_1
- Q1 pad 1: Net-(D1-A) -> Net-(Q1-G)
- Q1 pad 2: Net-(Q1-G) -> GND
- Q1 pad 3: unconnected-(Q1-S-Pad3) -> /DC supplies/PWR_3V3_2
- R1 pad 1: unconnected-(R1-Pad1) -> +3V3
- R1 pad 2: Net-(Q1-G) -> Net-(U3-~{PG})

Commit message: Commit de propreté
Parts:
- removed D1: D_Schottky, Diode_SMD:D_SMA
- added C4: 33µF, Capacitor_SMD:C_1206_3216Metric, F.Cu at (90.0, 47.4)
- added R7: 56K, Resistor_SMD:R_1206_3216Metric, F.Cu at (81.1, 48.6)
- C1: footprint Capacitor_THT:CP_Radial_D6.3mm_P2.50mm -> Capacitor_THT:CP_Radial_D5.0mm_P2.00mm
- J1, J6: footprint Connector_Wago:Wago_734-133_1x03_P3.50mm_Vertical -> Borniers:5442183
- J2: footprint Connector_Wuerth:Wuerth_WR-WTB_64800211622_1x02_P1.50mm_Vertical -> Borniers:5442170
- J3, J4, J5: footprint Connector_Wago:Wago_734-132_1x02_P3.50mm_Vertical -> Borniers:5442170
- J7: footprint Connector_JAE:JAE_LY20-14P-DT1_2x07_P2.00mm_Vertical -> Borniers:M80-85312YY
- moved R3 150.4 mm to (82.0, 105.8), turned to 90 degrees
- moved R4 145.7 mm to (86.0, 105.8), turned to 90 degrees
- moved U4 144.7 mm to (85.6, 120.4), turned to 90 degrees
- moved R5 141.0 mm to (90.0, 105.8), turned to 90 degrees
- moved R2 140.5 mm to (86.8, 71.5)
- moved Q3 139.6 mm to (97.6, 100.1), turned to 90 degrees
- moved Q6 136.7 mm to (96.4, 81.6), turned to -90 degrees
- moved U2 136.6 mm to (89.4, 136.2), turned to 90 degrees
- moved R6 136.5 mm to (93.8, 105.8), turned to 90 degrees
- moved J7 135.5 mm to (87.0, 91.9), turned to 180 degrees
- moved U6 133.0 mm to (92.6, 57.5), turned to -90 degrees
- moved Q2 131.6 mm to (82.4, 100.1), turned to 90 degrees
- moved U5 130.1 mm to (96.4, 120.4), turned to 90 degrees
- moved Q4 122.7 mm to (90.0, 100.1), turned to 90 degrees
- moved U7 121.8 mm to (98.3, 137.5), turned to 90 degrees
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- renumbered U3 to locked
Connections:
- U1 pad 16: /Power supply and relays/Relay_4 -> /Power supply and relays/Relay_2
- U1 pad 19: /Power supply and relays/Relay_2 -> /Power supply and relays/Relay_1
- U1 pad 20: /Power supply and relays/Relay_1 -> /Power supply and relays/Relay_4
- U6 pad 8: unconnected-(U6-SYNC-Pad8) -> Net-(U6-SYNC)
- U6 pad 9: unconnected-(U6-MUTE-Pad9) -> Net-(U6-MUTE)
Routing:
- net +5V: track 0.00 -> 389.2 mm, vias 0 -> 4
- net GND: track 0.00 -> 374.4 mm, vias 0 -> 12
- net NEUT: track 0.00 -> 219.5 mm
- net LINE: track 0.00 -> 202.4 mm
- net /DC supplies/MOSI: track 0.00 -> 199.6 mm, vias 0 -> 8
- net /DC supplies/SCLK: track 0.00 -> 153.8 mm, vias 0 -> 4
- net /DC supplies/~{RESET_IO}: track 0.00 -> 146.3 mm, vias 0 -> 6
- net +3V3: track 0.00 -> 130.9 mm
- net /MCU/~{CS_RELAY}: track 0.00 -> 117.4 mm, vias 0 -> 4
- net /DC supplies/CS_PWR_DC: track 0.00 -> 108.4 mm, vias 0 -> 2
- net /Power supply and relays/Relay_1: track 0.00 -> 94.8 mm
- net Earth: track 0.00 -> 91.6 mm
- net /DC supplies/LATCH: track 0.00 -> 86.6 mm, vias 0 -> 2
- net /Power supply and relays/Relay_4: track 0.00 -> 77.8 mm
- net Net-(Q8-G): track 0.00 -> 65.0 mm, vias 0 -> 2
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- added copper zone on B.Cu, net GND
- added copper zone on F.Cu, net GND
- added copper zone on B.Cu, net NEUT
- added copper zone on F.Cu, net NEUT
Other:
- board outline added: 184 x 114 mm
- board text added: "/!\ Danger 230 V"
- board text added: "BOT"
- board text added: "TOP"
- board text added: "Ver 1.1"

Commit message: Doc api
Parts:
- added H1: MountingHole, MountingHole:MountingHole_4.3mm_M4, F.Cu at (225.0, 72.8)
- added H2: MountingHole, MountingHole:MountingHole_4.3mm_M4, F.Cu at (225.0, 117.2)
- added H3: MountingHole, MountingHole:MountingHole_4.3mm_M4, F.Cu at (71.5, 72.8)
- added H4: MountingHole, MountingHole:MountingHole_4.3mm_M4, F.Cu at (71.5, 117.2)
- added REF**: Symbol_HighVoltage_Triangle_8x7mm_Copper, Symbol:Symbol_HighVoltage_Triangle_8x7mm_Copper, F.Cu at (205.7, 94.0)
- PS2: value MPM-45 -> MPM-30-5; footprint Multiprise pilotée:Converter_ACDC_MeanWell_MPM-45-xx_THT -> Multiprise pilotée:Converter_ACDC_MeanWell_MPM-30-xx_THT
- moved PS2 13.7 mm to (199.7, 113.9)
- moved J5 11.7 mm to (177.0, 62.0)
- moved J4 11.0 mm to (172.0, 127.0)
- moved J2 8.04 mm to (201.0, 62.0)
- moved K1 7.50 mm to (134.0, 57.2)
- moved K4 7.45 mm to (134.0, 71.2)
- moved K3 7.31 mm to (134.0, 125.7)
- moved J3 7.04 mm to (196.0, 127.0)
- moved K2 7.00 mm to (134.0, 139.7)
Connections:
- net Net-(J2-Pin_1) renamed /Power supply and relays/R1_L
- net Net-(J2-Pin_2) renamed /Power supply and relays/R1_N
- net Net-(J3-Pin_1) renamed /Power supply and relays/R2_L
- net Net-(J3-Pin_2) renamed /Power supply and relays/R2_N
- net Net-(J4-Pin_1) renamed /Power supply and relays/R3_L
- net Net-(J4-Pin_2) renamed /Power supply and relays/R3_N
- net Net-(J5-Pin_1) renamed /Power supply and relays/R4_L
- net Net-(J5-Pin_2) renamed /Power supply and relays/R4_N
- U1 pad 2: unconnected-(U1-~{SET}-Pad2) -> +5V
Routing:
- net LINE: track 202.4 -> 253.5 mm
- net NEUT: track 219.5 -> 263.0 mm
- net +5V: track 389.2 -> 346.2 mm, vias 4 -> 5
- net /Power supply and relays/Relay_1: track 94.8 -> 71.5 mm, vias 0 -> 1
- net /Power supply and relays/Relay_4: track 77.8 -> 100.0 mm, vias 0 -> 1
- net GND: track 374.4 -> 389.4 mm
- net /Power supply and relays/R1_L: track 52.6 -> 67.5 mm
- net /Power supply and relays/R2_N: track 52.2 -> 66.6 mm
- net /Power supply and relays/Relay_2: track 43.8 -> 30.1 mm
- net /Power supply and relays/R4_N: track 23.0 -> 13.7 mm
- net /Power supply and relays/R4_L: track 35.5 -> 26.8 mm
- net /Power supply and relays/R3_L: track 21.9 -> 13.6 mm
- net /Power supply and relays/Relay_3: track 25.0 -> 17.4 mm
- net /Power supply and relays/R3_N: track 33.8 -> 27.4 mm
- net Earth: track 91.6 -> 94.0 mm
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- removed copper zone on B.Cu, net NEUT
- removed copper zone on F.Cu, net NEUT
Other:
- board size 184 x 114 mm -> 184 x 107.5 mm
- board text added: "AC/L"
- board text added: "AC/N"
- board text added: "L"
- board text added: "N"
- board text added: "V+"
- board text added: "V-"
- board text added: "Ver 1.2"
- board text removed: "Ver 1.1"

Commit message: Ajout du projet asservissement de balle en python
Changed lines of the file:
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@@
     (pad_to_mask_clearance 0)
     (pcbplotparams
-      (layerselection 0x0000000_fffffffe)
+      (layerselection 0x00000ff_ffffffff)
       (plot_on_all_layers_selection 0x0001000_00000000)
       (disableapertmacros false)
@@
       (sketchpadsonfab false)
       (subtractmaskfromsilk false)
-      (outputformat 4)
-      (mirror true)
-      (drillshape 2)
+      (outputformat 1)
+      (mirror false)
+      (drillshape 0)
       (scaleselection 1)
-      (outputdirectory "PDF/")
+      (outputdirectory "Gerber/")
     )
   )
@@
     (fp_line (start 5.625 5) (end 4.625 5)
       (stroke (width 0.1) (type solid)) (layer "F.Fab"))
-    (pad "1" smd roundrect locked (at -7.65 -3.4 270) (size 4.6 1.1) (layers "F.Cu" "F.Paste" "F.Mask") (roundrect_rratio 0.227273)
+    (pad "1" smd roundrect locked (at -7.65 -3.4 270) (size 4.6 1.1) (layers "F.Cu" "F.Paste" "F.Mask") (roundrect_rratio 0.2272727273)
       (net 5 "GND") (pinfunction "~{EN}") (pintype "input"))
-    (pad "2" smd roundrect locked (at -7.65 -1.7 270) (size 4.6 1.1) (layers "F.Cu" "F.Paste" "F.Mask") (roundrect_rratio 0.227273)
+    (pad "2" smd roundrect locked (at -7.65 -1.7 270) (size 4.6 1.1) (layers "F.Cu" "F.Paste" "F.Mask") (roundrect_rratio 0.2272727273)
       (net 6 "+5V") (pinfunction "IN") (pintype "power_in"))
-    (pad "3" smd roundrect locked (at -7.65 0 270) (size 4.6 1.1) (layers "F.Cu" "F.Paste" "F.Mask") (roundrect_rratio 0.227273)
+    (pad "3" smd roundrect locked (at -7.65 0 270) (size 4.6 1.1) (layers "F.Cu" "F.Paste" "F.Mask") (roundrect_rratio 0.2272727273)
       (net 5 "GND") (pinfunction "GND") (pintype "power_in"))
-    (pad "4" smd roundrect locked (at -7.65 1.7 270) (size 4.6 1.1) (layers "F.Cu" "F.Paste" "F.Mask") (roundrect_rratio 0.227273)
+    (pad "4" smd roundrect locked (at -7.65 1.7 270) (size 4.6 1.1) (layers "F.Cu" "F.Paste" "F.Mask") (roundrect_rratio 0.2272727273)
       (net 3 "+3V3") (pinfunction "OUT") (pintype "power_out"))
-    (pad "5" smd roundrect locked (at -7.65 3.4 270) (size 4.6 1.1) (layers "F.Cu" "F.Paste" "F.Mask") (roundrect_rratio 0.227273)
+    (pad "5" smd roundrect locked (at -7.65 3.4 270) (size 4.6 1.1) (layers "F.Cu" "F.Paste" "F.Mask") (roundrect_rratio 0.2272727273)
       (net 44 "Net-(U3-~{PG})") (pinfunction "~{PG}") (pintype "open_collector"))
-    (pad "6" smd roundrect locked (at -0.925 -2.775 270) (size 4.55 5.25) (layers "F.Cu" "F.Paste") (roundrect_rratio 0.054945))
-    (pad "6" smd roundrect locked (at -0.925 2.775 270) (size 4.55 5.25) (layers "F.Cu" "F.Paste") (roundrect_rratio 0.054945))
-    (pad "6" smd roundrect locked (at 1.5 0 270) (size 9.4 10.8) (layers "F.Cu" "F.Mask") (roundrect_rratio 0.026596))
-    (pad "6" smd roundrect locked (at 3.925 -2.775 270) (size 4.55 5.25) (layers "F.Cu" "F.Paste") (roundrect_rratio 0.054945))
-    (pad "6" smd roundrect locked (at 3.925 2.775 270) (size 4.55 5.25) (layers "F.Cu" "F.Paste") (roundrect_rratio 0.054945))
+    (pad "6" smd roundrect locked (at -0.925 -2.775 270) (size 4.55 5.25) (layers "F.Cu" "F.Paste") (roundrect_rratio 0.05494505495))
+    (pad "6" smd roundrect locked (at -0.925 2.775 270) (size 4.55 5.25) (layers "F.Cu" "F.Paste") (roundrect_rratio 0.05494505495))
+    (pad "6" smd roundrect locked (at 1.5 0 270) (size 9.4 10.8) (layers "F.Cu" "F.Mask") (roundrect_rratio 0.02659595745))
+    (pad "6" smd roundrect locked (at 3.925 -2.775 270) (size 4.55 5.25) (layers "F.Cu" "F.Paste") (roundrect_rratio 0.05494505495))
+    (pad "6" smd roundrect locked (at 3.925 2.775 270) (size 4.55 5.25) (layers "F.Cu" "F.Paste") (roundrect_rratio 0.05494505495))
     (model "${KICAD6_3DMODEL_DIR}/Package_TO_SOT_SMD.3dshapes/TO-263-5_TabPin6.wrl"
       (offset (xyz 0 0 0))
